Commit message: Added hokuyo mesh to both version. ROS1 is working with forwarding controller.

File: catkin_ws/src/rrbot_description/urdf/rrbot/rrbot.urdf.xacro (robot description, xacro)
@@ -109,4 +109,30 @@
         <link name="${prefix}tool_link">
         </link>
+        <joint name="${prefix}hokuyo_joint" type="fixed">
+          <axis xyz="0 1 0" />
+          <origin xyz="0 0 ${height3 - axel_offset/2}" rpy="0 0 0"/>
+          <parent link="${prefix}link2"/>
+          <child link="${prefix}hokuyo_link"/>
+        </joint>
+        <!-- Hokuyo Laser -->
+        <link name="${prefix}hokuyo_link">
+          <collision>
+            <origin xyz="0 0 0" rpy="0 0 0"/>
+            <geometry>
+              <box size="0.1 0.1 0.1"/>
+            </geometry>
+          </collision>
+          <visual>
+            <origin xyz="0 0 0" rpy="0 0 0"/>
+            <geometry>
+              <mesh filename="package://rrbot_description/meshes/hokuyo.dae"/>
+            </geometry>
+          </visual>
+          <inertial>
+            <mass value="1e-5" />
+            <origin xyz="0 0 0" rpy="0 0 0"/>
+            <inertia ixx="1e-6" ixy="0" ixz="0" iyy="1e-6" iyz="0" izz="1e-6" />
+          </inertial>
+        </link>
         <joint name="${prefix}camera_joint" type="fixed">
           <axis xyz="0 1 0" />
